File: keyboard.kicad_sch (KiCad schematic)
At the start: 22 parts, among them Q1 BSS138, Q2 BSS138, Q3 BSS138, Q4 BSS138, Q5 BSS138, Q6 BSS138, U4 ME6212C18M5G, U5 ME6212C28M5G

Commit message: footprint1
Parts:
- added JP1: SolderJumper_2_Open, Jumper:SolderJumper-2_P1.3mm_Open_RoundedPad1.0x1.5mm, symbol Jumper:SolderJumper_2_Open
- C14, C15: footprint (none) -> Capacitor_SMD:C_0603_1608Metric
- R11, R12, R13, R14, R15, R16, R17, R18, R19, R20, R21: footprint (none) -> Resistor_SMD:R_0603_1608Metric
- U6: value ~ -> BBQ20KBD; footprint (none) -> BM20B_0:HRS_BM20B_0.8_-40DS-0.4V_51_
Connections:
- net +3V3: now also JP1.1 (A)
- net at U6.24 (MIC_VDD): now also JP1.2 (B)
Changed lines of the file:
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@@
 	)
 	(junction
+		(at 149.86 76.2)
+		(diameter 0)
+		(color 0 0 0 0)
+	)
+	(junction
 		(at 49.53 140.97)
 		(diameter 0)
@@
 	(wire
 		(pts
-			(xy 149.86 81.28) (xy 149.86 69.85)
+			(xy 149.86 81.28) (xy 149.86 76.2)
 		)
 		(stroke
@@
 	(wire
 		(pts
+			(xy 149.86 76.2) (xy 152.4 76.2)
+		)
+		(stroke
+			(width 0)
+			(type default)
+		)
+	)
+	(wire
+		(pts
 			(xy 109.22 73.66) (xy 109.22 76.2)
 		)
@@
 	(wire
 		(pts
+			(xy 149.86 76.2) (xy 149.86 69.85)
+		)
+		(stroke
+			(width 0)
+			(type default)
+		)
+	)
+	(wire
+		(pts
 			(xy 49.53 29.21) (xy 49.53 30.48)
 		)
@@
 	(wire
 		(pts
+			(xy 160.02 76.2) (xy 161.29 76.2)
+		)
+		(stroke
+			(width 0)
+			(type default)
+		)
+	)
+	(wire
+		(pts
 			(xy 41.91 31.75) (xy 41.91 29.21)
 		)
@@
 			)
 		)
-		(property "Footprint" ""
+		(property "Footprint" "Resistor_SMD:R_0603_1608Metric"
 			(at 32.512 34.29 90)
 			(effects
@@
 		(on_board yes)
 		(dnp no)
-		(fields_autoplaced yes)
 		(property "Reference" "U6"
-			(at 176.53 64.77 0)
+			(at 183.388 66.802 0)
 			(effects
 				(font
@@
 			)
 		)
-		(property "Value" "~"
-			(at 176.53 67.31 0)
+		(property "Value" "BBQ20KBD"
+			(at 176.276 121.92 0)
 			(effects
 				(font
@@
 			)
 		)
-		(property "Footprint" ""
+		(property "Footprint" "BM20B_0:HRS_BM20B_0.8_-40DS-0.4V_51_"
 			(at 176.53 68.58 0)
 			(effects
@@
 			)
 		)
-		(property "Footprint" ""
+		(property "Footprint" "Resistor_SMD:R_0603_1608Metric"
 			(at 121.412 97.79 90)
 			(effects
@@
 			)
 		)
-		(property "Footprint" ""
+		(property "Footprint" "Resistor_SMD:R_0603_1608Metric"
 			(at 47.752 135.89 90)
 			(effects
@@
 			)
 		)
-		(property "Footprint" ""
+		(property "Footprint" "Resistor_SMD:R_0603_1608Metric"
 			(at 32.512 135.89 90)
 			(effects
@@
 			)
 		)
-		(property "Footprint" ""
+		(property "Footprint" "Resistor_SMD:R_0603_1608Metric"
 			(at 32.512 85.09 90)
 			(effects
@@
 			)
 		)
-		(property "Footprint" ""
+		(property "Footprint" "Resistor_SMD:R_0603_1608Metric"
 			(at 32.512 110.49 90)
 			(effects
@@
 			)
 		)
-		(property "Footprint" ""
+		(property "Footprint" "Resistor_SMD:R_0603_1608Metric"
 			(at 47.752 59.69 90)
 			(effects
@@
 	)
 	(symbol
+		(lib_id "Jumper:SolderJumper_2_Open")
+		(at 156.21 76.2 0)
+		(unit 1)
+		(exclude_from_sim yes)
+		(in_bom no)
+		(on_board yes)
+		(dnp no)
+		(fields_autoplaced yes)
+		(property "Reference" "JP1"
+			(at 156.21 69.85 0)
+			(effects
+				(font
+					(size 1.27 1.27)
+				)
+			)
+		)
+		(property "Value" "SolderJumper_2_Open"
+			(at 156.21 72.39 0)
+			(effects
+				(font
+					(size 1.27 1.27)
+				)
+				(hide yes)
+			)
+		)
+		(property "Footprint" "Jumper:SolderJumper-2_P1.3mm_Open_RoundedPad1.0x1.5mm"
+			(at 156.21 76.2 0)
+			(effects
+				(font
+					(size 1.27 1.27)
+				)
+				(hide yes)
+			)
+		)
+		(property "Datasheet" "~"
+			(at 156.21 76.2 0)
+			(effects
+				(font
+					(size 1.27 1.27)
+				)
+				(hide yes)
+			)
+		)
+		(property "Description" "Solder Jumper, 2-pole, open"
+			(at 156.21 76.2 0)
+			(effects
+				(font
+					(size 1.27 1.27)
+				)
+				(hide yes)
+			)
+		)
+		(pin "1"
+		)
+		(pin "2"
+		)
+		(instances
+			(project ""
+				(path "/9cb59c1c-3f16-4fc8-8e14-5089e3b6ad71/dad46d0a-22b9-4133-b417-9fdda3ca9b79"
+					(reference "JP1")
+					(unit 1)
+				)
+			)
+		)
+	)
+	(symbol
 		(lib_id "power:GND")
 		(at 133.35 100.33 0)
@@
 			)
 		)
-		(property "Footprint" ""
+		(property "Footprint" "Resistor_SMD:R_0603_1608Metric"
 			(at 47.752 34.29 90)
 			(effects
@@
 			)
 		)
-		(property "Footprint" ""
+		(property "Footprint" "Resistor_SMD:R_0603_1608Metric"
 			(at 47.752 110.49 90)
 			(effects
@@
 			)
 		)
-		(property "Footprint" ""
+		(property "Footprint" "Capacitor_SMD:C_0603_1608Metric"
 			(at 110.1852 50.8 0)
 			(effects
@@
 			)
 		)
-		(property "Footprint" ""
+		(property "Footprint" "Resistor_SMD:R_0603_1608Metric"
 			(at 47.752 85.09 90)
 			(effects
@@
 			)
 		)
-		(property "Footprint" ""
+		(property "Footprint" "Resistor_SMD:R_0603_1608Metric"
 			(at 32.512 59.69 90)
 			(effects
@@
 			)
 		)
-		(property "Footprint" ""
+		(property "Footprint" "Capacitor_SMD:C_0603_1608Metric"
 			(at 110.1852 83.82 0)
 			(effects

Commit message: PCB1
Connections:
- net GND: now also Q6.2 (S); no longer Q6.3 (D)
- net at U6.33 (LEDK), U6.35 (LEDK), U6.37 (LEDK): now also Q6.3 (D); no longer Q6.2 (S)
Changed lines of the file:
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@@
 		(pin "4"
+		)
+		(pin "38"
+		)
+		(pin "39"
 		)
 		(instances
@@
 		(lib_id "Transistor_FET:BSS138")
 		(at 130.81 92.71 0)
-		(mirror x)
 		(unit 1)
 		(exclude_from_sim no)
@@
 		(dnp no)
 		(property "Reference" "Q6"
-			(at 129.286 89.408 0)
+			(at 129.286 96.012 0)
 			(effects
 				(font
@@
 		)
 		(property "Footprint" "Package_TO_SOT_SMD:SOT-23"
-			(at 135.89 90.805 0)
+			(at 135.89 94.615 0)
 			(effects
 				(font
@@
 		)
 		(property "Datasheet" "https://www.onsemi.com/pub/Collateral/BSS138-D.PDF"
-			(at 135.89 88.9 0)
-			(effects
-				(font
+			(at 135.89 96.52 0)
+			(effects
+				(font
