File: my_bbq20.kicad_sch (KiCad schematic)
At the start: 17 parts, among them J1 USB_C_Receptacle_USB2.0_16P, U1 AP2112K-3.3

Commit message: sch1
Parts:
- added C12, C13: 12pF, symbol Device:C
- added J2: Conn_01x04, symbol Connector_Generic:Conn_01x04
- added J3: Conn_01x06, symbol Connector_Generic:Conn_01x06
- added R10, R8, R9: 4.7k, symbol Device:R
- added R22, R6: 1k, symbol Device:R
- added R3, R4: 27R, symbol Device:R
- added R5: 10k, symbol Device:R
- added R7: R, symbol Device:R
- added TP1, TP2, TP3, TP4, TP7: TestPoint, symbol Connector:TestPoint
- added U3: W25Q64JV, Package_SON:WSON-8-1EP_6x5mm_P1.27mm_EP3.4x4mm, symbol Memory_Flash_Extra:W25Q64JV
- added Y1: Crystal_GND24_Small, symbol Device:Crystal_GND24_Small
Connections:
- net +3V3: now also J2.2 (Pin_2), J3.1 (Pin_1), R10.1, R5.1, R7.1, R8.1, R9.1, U3.8 (VDD)
- net GND: now also C12.1, C13.1, J2.1 (Pin_1), J3.2 (Pin_2), U3.4 (GND), U3.9 (GND), Y1.2, Y1.4
- net USB_D+: now also R3.1
- net USB_D-: now also R4.1
- net COL1: now reaches U2.11 (GPIO8)
- net COL2: now reaches U2.12 (GPIO9)
- net COL3: now reaches U2.13 (GPIO10)
- net COL4: now reaches U2.14 (GPIO11)
- net COL5: now reaches U2.15 (GPIO12)
- net COL6: now reaches U2.16 (GPIO13)
- net BOOTSEL: now reaches U2.17 (GPIO14)
- net BOOTSEL: now also R22.1, TP1.1
- net INT: now reaches U2.2 (GPIO0)
- net INT: now also J3.6 (Pin_6), R8.2
- net at U2.20 (XIN): now also C12.2, Y1.3
- net at U2.21 (XOUT): now also R6.2
- net SWCLK: now reaches U2.24 (SWCLK)
- net SWCLK: now also TP3.1
- net SWDIO: now reaches U2.25 (SWD)
- net SWDIO: now also TP4.1
- net ~{RESET}: now reaches U2.26 (RUN)
- net ~{RESET}: now also R5.2, TP2.1
- net TP_RESET: now reaches U2.27 (GPIO16)
- net TP_SDA: now reaches U2.29 (GPIO18)
- net ROW1: now reaches U2.3 (GPIO1)
- net TX: now reaches U2.31 (GPIO20)
- net TX: now also TP7.1
- net TP_MOTION: now reaches U2.34 (GPIO22)
- net TP_SCL: now reaches U2.35 (GPIO23)
- net TP_SHUTDOWN: now reaches U2.36 (GPIO24)
- net BACKLIGHT: now reaches U2.37 (GPIO25)
- net MIC: now reaches U2.39 (GPIO27_ADC1)
- net ROW2: now reaches U2.4 (GPIO2)
- net SDA: now reaches U2.40 (GPIO28_ADC2)
- net SDA: now also J2.3 (Pin_3), J3.3 (Pin_3), R9.2
- net SCL: now reaches U2.41 (GPIO29_ADC3)
- net SCL: now also J2.4 (Pin_4), J3.4 (Pin_4), R10.2
- net at U2.46 (USB_DM): now also R4.2
- net at U2.47 (USB_DP): now also R3.2
- net ROW3: now reaches U2.5 (GPIO3)
- net QSPI_SD3: now reaches U2.51 (QSPI_SD3)
- net QSPI_SD3: now also U3.7 (~{HOLD}/IO3)
- net QSPI_SCLK: now reaches U2.52 (QSPI_SCLK)
- net QSPI_SCLK: now also U3.6 (SCK)
- net QSPI_SD0: now reaches U2.53 (QSPI_SD0)
- net QSPI_SD0: now also U3.5 (DI/IO0)
- net QSPI_SD2: now reaches U2.54 (QSPI_SD2)
- net QSPI_SD2: now also U3.3 (~{WP}/IO2)
- net QSPI_SD1: now reaches U2.55 (QSPI_SD1)
- net QSPI_SD1: now also U3.2 (DO/IO1)
- net ~{QSPI_CS}: now reaches U2.56 (QSPI_SS)
- net ~{QSPI_CS}: now also R22.2, R7.2, U3.1 (~{CS})
- net ROW4: now reaches U2.6 (GPIO4)
- net ROW5: now reaches U2.7 (GPIO5)
- net ROW6: now reaches U2.8 (GPIO6)
- net ROW7: now reaches U2.9 (GPIO7)
- new net: C13.2, R6.1, Y1.1
- no-connect marks 2 -> 9
Other:
- added sheet Keyborad (keyboard.kicad_sch)

Commit message: footprint1
Parts:
- C1, C10, C11, C12, C13, C2, C3, C4, C5, C6, C7, C8, C9: footprint (none) -> Capacitor_SMD:C_0603_1608Metric
- D1: footprint (none) -> Diode_SMD:D_SOD-323
- J1: footprint (none) -> Connector_USB:USB_C_Receptacle_HRO_TYPE-C-31-M-12
- J2: footprint (none) -> Connector_JST:JST_GH_SM04B-GHS-TB_1x04-1MP_P1.25mm_Horizontal
- J3: footprint (none) -> Connector_PinHeader_2.54mm:PinHeader_1x06_P2.54mm_Horizontal
- R1, R10, R2, R22, R3, R4, R5, R6, R8, R9: footprint (none) -> Resistor_SMD:R_0603_1608Metric
- R7: value R -> 10k; footprint (none) -> Resistor_SMD:R_0603_1608Metric
- TP1, TP2, TP3, TP4, TP7: footprint (none) -> TestPoint:TestPoint_Pad_D1.5mm
- U2: footprint (none) -> RP2040:QFN40P700X700X90-57N
- U3: footprint Package_SON:WSON-8-1EP_6x5mm_P1.27mm_EP3.4x4mm -> Package_SO:SOIC-8_5.275x5.275mm_P1.27mm
- Y1: footprint (none) -> Crystal:Crystal_SMD_2520-4Pin_2.5x2.0mm
Changed lines of the file:
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@@
 			)
 		)
-		(property "Footprint" ""
+		(property "Footprint" "Diode_SMD:D_SOD-323"
 			(at 39.37 95.25 90)
 			(effects
@@
 			)
 		)
-		(property "Footprint" ""
+		(property "Footprint" "Resistor_SMD:R_0603_1608Metric"
 			(at 63.5 42.418 90)
 			(effects
@@
 			)
 		)
-		(property "Footprint" ""
+		(property "Footprint" "Resistor_SMD:R_0603_1608Metric"
 			(at 93.98 70.358 90)
 			(effects
@@
 			)
 		)
-		(property "Footprint" ""
+		(property "Footprint" "Capacitor_SMD:C_0603_1608Metric"
 			(at 104.14 48.5648 0)
 			(effects
@@
 			)
 		)
-		(property "Footprint" ""
+		(property "Footprint" "Resistor_SMD:R_0603_1608Metric"
 			(at 135.382 152.4 90)
 			(effects
@@
 			)
 		)
-		(property "Footprint" ""
+		(property "Footprint" "Connector_PinHeader_2.54mm:PinHeader_1x06_P2.54mm_Horizontal"
 			(at 125.73 166.37 0)
 			(effects
@@
 			)
 		)
-		(property "Footprint" ""
+		(property "Footprint" "Capacitor_SMD:C_0603_1608Metric"
 			(at 104.14 59.9948 0)
 			(effects
@@
 			)
 		)
-		(property "Footprint" ""
+		(property "Footprint" "TestPoint:TestPoint_Pad_D1.5mm"
 			(at 88.9 116.84 0)
 			(effects
@@
 			)
 		)
-		(property "Footprint" ""
+		(property "Footprint" "Capacitor_SMD:C_0603_1608Metric"
 			(at 128.5748 25.4 0)
 			(effects
@@
 			)
 		)
-		(property "Footprint" ""
+		(property "Footprint" "TestPoint:TestPoint_Pad_D1.5mm"
 			(at 167.64 100.33 0)
 			(effects
@@
 			)
 		)
-		(property "Footprint" ""
+		(property "Footprint" "Connector_JST:JST_GH_SM04B-GHS-TB_1x04-1MP_P1.25mm_Horizontal"
 			(at 92.71 166.37 0)
 			(effects
@@
 			)
 		)
-		(property "Footprint" ""
+		(property "Footprint" "Capacitor_SMD:C_0603_1608Metric"
 			(at 104.14 40.9448 0)
 			(effects
@@
 			)
 		)
-		(property "Footprint" ""
+		(property "Footprint" "Resistor_SMD:R_0603_1608Metric"
 			(at 83.312 58.42 90)
 			(effects
@@
 			)
 		)
-		(property "Footprint" ""
+		(property "Footprint" "Resistor_SMD:R_0603_1608Metric"
 			(at 131.572 152.4 90)
 			(effects
@@
 			)
 		)
-		(property "Footprint" ""
+		(property "Footprint" "Capacitor_SMD:C_0603_1608Metric"
 			(at 104.14 56.1848 0)
 			(effects
@@
 			)
 		)
-		(property "Footprint" ""
+		(property "Footprint" "Capacitor_SMD:C_0603_1608Metric"
 			(at 104.14 52.3748 0)
 			(effects
@@
 			)
 		)
-		(property "Footprint" ""
+		(property "Footprint" "Resistor_SMD:R_0603_1608Metric"
 			(at 141.732 152.4 90)
 			(effects
@@
 			)
 		)
-		(property "Footprint" ""
+		(property "Footprint" "RP2040:QFN40P700X700X90-57N"
 			(at 128.27 34.29 0)
 			(effects
@@
 			)
 		)
-		(property "Footprint" ""
+		(property "Footprint" "Capacitor_SMD:C_0603_1608Metric"
 			(at 26.3652 119.38 0)
 			(effects
@@
 			)
 		)
-		(property "Footprint" ""
+		(property "Footprint" "Connector_USB:USB_C_Receptacle_HRO_TYPE-C-31-M-12"
 			(at 44.45 48.26 0)
 			(effects
@@
 			)
 		)
-		(property "Footprint" ""
+		(property "Footprint" "TestPoint:TestPoint_Pad_D1.5mm"
 			(at 81.28 82.55 0)
 			(effects
@@
 			)
 		)
-		(property "Footprint" ""
+		(property "Footprint" "Crystal:Crystal_SMD_2520-4Pin_2.5x2.0mm"
 			(at 86.36 105.41 0)
 			(effects
@@
 			)
 		)
-		(property "Footprint" ""
+		(property "Footprint" "Capacitor_SMD:C_0603_1608Metric"
 			(at 104.14 44.7548 0)
 			(effects
@@
 			)
 		)
-		(property "Footprint" ""
+		(property "Footprint" "Capacitor_SMD:C_0603_1608Metric"
 			(at 124.7648 25.4 0)
 			(effects
@@
 			)
 		)
-		(property "Footprint" ""
+		(property "Footprint" "Capacitor_SMD:C_0603_1608Metric"
 			(at 132.3848 25.4 0)
 			(effects
@@
 			)
 		)
-		(property "Footprint" ""
+		(property "Footprint" "TestPoint:TestPoint_Pad_D1.5mm"
 			(at 73.66 59.69 0)
 			(effects
@@
 			)
 		)
-		(property "Value" "R"
+		(property "Value" "10k"
 			(at 60.96 148.5899 0)
 			(effects
@@
 			)
 		)
-		(property "Footprint" ""
+		(property "Footprint" "Resistor_SMD:R_0603_1608Metric"
 			(at 56.642 147.32 90)
 			(effects
@@
 			)
 		)
-		(property "Footprint" ""
+		(property "Footprint" "TestPoint:TestPoint_Pad_D1.5mm"
 			(at 88.9 114.3 0)
 			(effects
@@
 			)
 		)
-		(property "Footprint" ""
+		(property "Footprint" "Resistor_SMD:R_0603_1608Metric"
 			(at 99.06 112.268 90)
 			(effects
@@
 			)
 		)
-		(property "Footprint" ""
+		(property "Footprint" "Resistor_SMD:R_0603_1608Metric"
 			(at 63.5 39.878 90)
 			(effects
@@
 			)
 		)
-		(property "Footprint" ""
+		(property "Footprint" "Resistor_SMD:R_0603_1608Metric"
 			(at 90.17 79.248 90)
 			(effects
@@
 			)
 		)
-		(property "Footprint" "Package_SON:WSON-8-1EP_6x5mm_P1.27mm_EP3.4x4mm"
+		(property "Footprint" "Package_SO:SOIC-8_5.275x5.275mm_P1.27mm"
 			(at 44.45 172.72 0)
 			(effects
@@
 			)
 		)
-		(property "Footprint" ""
+		(property "Footprint" "Resistor_SMD:R_0603_1608Metric"
 			(at 93.98 72.898 90)
 			(effects
@@
 			)
 		)
-		(property "Footprint" ""
+		(property "Footprint" "Capacitor_SMD:C_0603_1608Metric"
 			(at 80.01 109.5248 0)
 			(effects
@@
 			)
 		)
-		(property "Footprint" ""
+		(property "Footprint" "Capacitor_SMD:C_0603_1608Metric"
 			(at 51.7652 119.38 0)
 			(effects
@@
 			)
 		)
-		(property "Footprint" ""
+		(property "Footprint" "Capacitor_SMD:C_0603_1608Metric"
 			(at 80.01 99.3648 0)
 			(effects

Commit message: PCB1
Parts:
- U3: footprint Package_SO:SOIC-8_5.275x5.275mm_P1.27mm -> Package_SON:WSON-8-1EP_6x5mm_P1.27mm_EP3.4x4mm
Changed lines of the file:
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@@
 			)
 		)
-		(property "Footprint" "Package_SO:SOIC-8_5.275x5.275mm_P1.27mm"
+		(property "Footprint" "Package_SON:WSON-8-1EP_6x5mm_P1.27mm_EP3.4x4mm"
 			(at 44.45 172.72 0)
 			(effects
@@
 		(pin "8"
 		)
-		(pin "9"
-		)
 		(pin "1"
 		)
@@
 		(pin "4"
 		)
+		(pin "9"
+		)
 		(instances

Commit message: PCB Lay
Parts:
- added TP5, TP6: TestPoint, TestPoint:TestPoint_Pad_D1.5mm, symbol Connector:TestPoint
Connections:
- net +3V3: now also TP6.1
- net GND: now also TP5.1

Commit message: PCB2
Parts:
- J3: footprint Connector_PinHeader_2.54mm:PinHeader_1x06_P2.54mm_Horizontal -> my_footprint:Pmod_PinHeader_1x06_P2.54mm_Horizontal
- U3: footprint Package_SON:WSON-8-1EP_6x5mm_P1.27mm_EP3.4x4mm -> my_footprint:my_WSON-8-1EP_6x5mm_P1.27mm_EP3.4x4mm
Connections:
- net BOOTSEL: now also U2.13 (GPIO10); no longer U2.17 (GPIO14)
- net COL3: now also U2.17 (GPIO14); no longer U2.13 (GPIO10)
- net COL4: now also U2.16 (GPIO13); no longer U2.14 (GPIO11)
- net COL6: now also U2.14 (GPIO11); no longer U2.16 (GPIO13)
- net GND: no longer U3.9 (GND)
Changed lines of the file:
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@@
 		)
 	)
-	(label "COL7"
+	(label "COL3"
 		(at 156.21 80.01 0)
 		(effects
@@
 		)
 	)
-	(label "COL6"
+	(label "COL4"
 		(at 156.21 77.47 0)
 		(effects
@@
 		)
 	)
-	(label "COL4"
+	(label "COL6"
 		(at 156.21 72.39 0)
 		(effects
@@
 		)
 	)
-	(label "COL3"
+	(label "COL7"
 		(at 156.21 69.85 0)
 		(effects
@@
 			)
 		)
-		(property "Footprint" "Connector_PinHeader_2.54mm:PinHeader_1x06_P2.54mm_Horizontal"
+		(property "Footprint" "my_footprint:Pmod_PinHeader_1x06_P2.54mm_Horizontal"
 			(at 125.73 166.37 0)
 			(effects
@@
 			)
 		)
-		(property "Footprint" "Package_SON:WSON-8-1EP_6x5mm_P1.27mm_EP3.4x4mm"
+		(property "Footprint" "my_footprint:my_WSON-8-1EP_6x5mm_P1.27mm_EP3.4x4mm"
 			(at 44.45 172.72 0)
 			(effects
@@
 		(pin "4"
 		)
-		(pin "9"
-		)
 		(instances
