File: my_bbq20.kicad_pcb (KiCad board)
At the start: 2 copper layers, 60 parts, among them J1 USB_C_Receptacle_USB2.0_16P, J2 Conn_01x04, J3 Conn_01x06, Q1 BSS138, Q2 BSS138, Q3 BSS138, Q4 BSS138, Q5 BSS138, Q6 BSS138, U1 AP2112K-3.3, U3 W25Q64JV, U4 ME6212C18M5G, U5 ME6212C28M5G, U6 BBQ20KBD, Y1 Crystal_GND24_Small

Commit message: PCB Lay
Parts:
- added 3V3: TestPoint, TestPoint:TestPoint_Pad_D1.5mm, B.Cu at (111.0, 91.2)
- added GND: TestPoint, TestPoint:TestPoint_Pad_D1.5mm, B.Cu at (102.5, 91.2)
- moved U1 72.1 mm to (84.9, 61.5)
- moved D1 67.6 mm to (84.8, 58.8)
- moved U5 62.9 mm to (76.2, 66.0)
- moved JP1 62.3 mm to (74.3, 60.0)
- moved U4 55.8 mm to (76.2, 69.5)
- moved C1 55.5 mm to (87.7, 61.6), turned to -90 degrees
- moved C6 52.8 mm to (88.9, 76.7), turned to 0 degrees
- moved R2 49.7 mm to (96.5, 60.6), turned to -90 degrees
- moved R1 49.1 mm to (93.4, 60.6), turned to -90 degrees
- moved C15 47.8 mm to (73.4, 66.2), turned to -90 degrees
- moved C14 46.5 mm to (73.4, 69.7), turned to -90 degrees
- moved C4 42.5 mm to (102.3, 73.2)
- moved R5 41.7 mm to (90.2, 83.0), turned to 90 degrees
- moved C5 41.7 mm to (102.3, 76.7)
- moved C7 41.4 mm to (82.0, 61.5)
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- renumbered TP1 to BOOT, TP3 to CLK, TP4 to IO, TP2 to RST, TP7 to TX

Commit message: PCB2
Parts:
- J3: footprint Connector_PinHeader_2.54mm:PinHeader_1x06_P2.54mm_Horizontal -> my_footprint:Pmod_PinHeader_1x06_P2.54mm_Horizontal
- U3: footprint Package_SON:WSON-8-1EP_6x5mm_P1.27mm_EP3.4x4mm -> my_footprint:my_WSON-8-1EP_6x5mm_P1.27mm_EP3.4x4mm
- moved J3 10.5 mm to (116.9, 48.4), turned to 180 degrees
- moved C1 2.33 mm to (87.3, 63.9)
- moved C7 2.33 mm to (81.7, 63.8)
- moved D1 2.33 mm to (84.5, 61.0)
- moved U1 2.33 mm to (84.5, 63.8)
- moved J2 1.53 mm to (79.8, 51.9)
- moved U3 1.33 mm to (105.1, 68.2)
- moved R22 1.33 mm to (111.4, 67.2)
- moved R7 1.33 mm to (109.9, 67.2)
- moved R8 1.33 mm to (112.9, 67.2)
- moved C11 0.56 mm to (98.4, 68.7), turned to 90 degrees
- moved C8 0.56 mm to (96.9, 68.7)
- moved C9 0.56 mm to (92.4, 68.7)
- moved R3 0.56 mm to (95.4, 68.7)
- moved R4 0.56 mm to (93.9, 68.7)
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- renumbered BOOT to TP1, RST to TP2, CLK to TP3, IO to TP4, GND to TP5, 3V3 to TP6, TX to TP7
Connections:
- U2 pad 13: /COL3 -> /BOOTSEL
- U2 pad 14: /COL4 -> /COL6
- U2 pad 16: /COL6 -> /COL4
- U2 pad 17: /BOOTSEL -> /COL3
Routing:
- net +3V3: track 0.00 -> 163.7 mm, vias 0 -> 17
- net /COL3: track 0.00 -> 83.0 mm, vias 0 -> 1
- net /COL4: track 0.00 -> 80.1 mm, vias 0 -> 1
- net /COL5: track 0.00 -> 77.3 mm, vias 0 -> 1
- net /COL6: track 0.00 -> 73.1 mm, vias 0 -> 1
- net /BOOTSEL: track 0.00 -> 70.8 mm, vias 0 -> 1
- net /COL2: track 0.00 -> 69.3 mm, vias 0 -> 1
- net /COL1: track 0.00 -> 68.0 mm, vias 0 -> 1
- net /ROW7: track 0.00 -> 63.2 mm, vias 0 -> 1
- net /ROW6: track 0.00 -> 61.8 mm, vias 0 -> 1
- net /ROW5: track 0.00 -> 60.4 mm, vias 0 -> 1
- net /ROW4: track 0.00 -> 59.1 mm, vias 0 -> 1
- net /ROW3: track 0.00 -> 57.7 mm, vias 0 -> 1
- net /ROW2: track 0.00 -> 56.3 mm, vias 0 -> 1
- net /ROW1: track 0.00 -> 54.8 mm, vias 0 -> 1
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Other:
- board outline added: 75 x 54 mm

Commit message: pcb Cu
Parts:
- moved J2 1.75 mm to (78.0, 51.9)
- moved JP1 0.30 mm to (74.7, 60.0)
Routing:
- net /SDA: track 0.00 -> 74.9 mm, vias 0 -> 2
- net /SCL: track 0.00 -> 73.5 mm
- net /BOOTSEL: track 70.8 -> 113.1 mm, vias 1 -> 5
- net +3V3: track 163.7 -> 201.7 mm, vias 17 -> 18
- net /MIC: track 2.98 -> 34.0 mm, vias 0 -> 1
- net /SWCLK: track 0.00 -> 23.8 mm, vias 0 -> 2
- net /TX: track 0.00 -> 17.4 mm, vias 0 -> 2
- net /SWDIO: track 0.00 -> 15.7 mm, vias 0 -> 2
- net Net-(JP1-B): track 0.00 -> 11.5 mm, vias 0 -> 1
- net /~{RESET}: track 5.62 -> 15.1 mm, vias 0 -> 1
- net +1V8: track 39.6 -> 48.3 mm
- net GND: track 0.00 -> 2.34 mm, vias 0 -> 1
- net /~{QSPI_CS}: track 18.1 -> 20.4 mm
- net (no net): vias 3 -> 0
- added copper zone on B.Cu, net GND
- added copper zone on F.Cu, net GND

Commit message: PCB 3
Parts:
- J3: value Conn_01x06 -> PMOD
- renumbered TP6 to 3V3, TP1 to BOOT, TP3 to CLK, TP5 to GND, J2 to I2C, TP4 to IO, TP2 to RST, TP7 to TX, J1 to USB
Routing:
- net /~{QSPI_CS}: track 20.4 -> 19.1 mm
- net /QSPI_SD1: track 15.4 -> 14.1 mm
- net /COL3: vias 1 -> 3
- net GND: vias 1 -> 33
Other:
- outline, holes or cut-outs redrawn

Commit message: DRC1
Routing:
- net GND: vias 33 -> 36
Other:
- outline, holes or cut-outs redrawn
Changed lines of the file:
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@@
 		(tags "test point SMD pad")
 		(property "Reference" "RST"
-			(at -4.2 0.066667 270)
+			(at -4.2 0.066667 -90)
 			(layer "B.SilkS")
 			(effects
@@
 	)
 	(gr_line
+		(start 69.75 58.5)
+		(end 60.75 58.5)
+		(stroke
+			(width 0.05)
+			(type default)
+		)
+		(layer "Edge.Cuts")
+	)
+	(gr_line
 		(start 130.5 52.5)
 		(end 130.5 92.5)
@@
 	)
 	(gr_arc
+		(start 69.75 53.5)
+		(mid 70.28033 53.71967)
+		(end 70.5 54.25)
+		(stroke
+			(width 0.05)
+			(type default)
+		)
+		(layer "Edge.Cuts")
+	)
+	(gr_arc
 		(start 60.15 77.7)
 		(mid 59.867157 77.582843)
@@
 		(layer "Edge.Cuts")
 	)
+	(gr_arc
+		(start 70.5 57.75)
+		(mid 70.28033 58.28033)
+		(end 69.75 58.5)
+		(stroke
+			(width 0.05)
+			(type default)
+		)
+		(layer "Edge.Cuts")
+	)
 	(gr_line
 		(start 60.15 77.7)
@@
 		(layer "Edge.Cuts")
 	)
+	(gr_arc
+		(start 60.75 58.5)
+		(mid 60.21967 58.28033)
+		(end 60 57.75)
+		(stroke
+			(width 0.05)
+			(type default)
+		)
+		(layer "Edge.Cuts")
+	)
+	(gr_line
+		(start 70.5 54.25)
+		(end 70.5 57.75)
+		(stroke
+			(width 0.05)
+			(type default)
+		)
+		(layer "Edge.Cuts")
+	)
 	(gr_line
 		(start 55.5 92.5)
@@
 		(layer "Edge.Cuts")
 	)
+	(gr_line
+		(start 60.75 53.5)
+		(end 69.75 53.5)
+		(stroke
+			(width 0.05)
+			(type default)
+		)
+		(layer "Edge.Cuts")
+	)
 	(gr_arc
 		(start 130.5 92.5)
@@
 		(layer "Edge.Cuts")
 	)
+	(gr_line
+		(start 60 57.75)
+		(end 60 54.25)
+		(stroke
+			(width 0.05)
+			(type default)
+		)
+		(layer "Edge.Cuts")
+	)
+	(gr_arc
+		(start 60 54.25)
+		(mid 60.21967 53.71967)
+		(end 60.75 53.5)
+		(stroke
+			(width 0.05)
+			(type default)
+		)
+		(layer "Edge.Cuts")
+	)
 	(segment
 		(start 92.23 56.545)
@@
 	)
 	(via
+		(at 79.5 66.5)
+		(size 0.6)
+		(drill 0.3)
+		(layers "F.Cu" "B.Cu")
+		(free yes)
+		(net 2)
+	)
+	(via
 		(at 103.15 79.3)
 		(size 0.6)
@@
 	)
 	(via
+		(at 65.25 70.75)
+		(size 0.6)
+		(drill 0.3)
+		(layers "F.Cu" "B.Cu")
+		(free yes)
+		(net 2)
+	)
+	(via
 		(at 120.5 64.6)
 		(size 0.8)
@@
 		(layers "F.Cu" "B.Cu")
 		(free yes)
+		(net 2)
+	)
+	(via
+		(at 79.5 69.75)
+		(size 0.6)
+		(drill 0.3)
+		(layers "F.Cu" "B.Cu")
+		(free yes)

Commit message: DRC2
Routing:
- net +2V8: track 13.8 -> 13.2 mm
